Commit message: Parte 2 (Localizacion) + fix castor + capturas de entrega
NUEVOS ARCHIVOS:
- launch/localization.launch.py: simulacion + map_server + amcl bajo un
  lifecycle_manager (map_server primero, amcl despues porque necesita el
  mapa ya publicado)
- config/localization.yaml: config de ambos nodos. map_server carga el
  mapa; amcl es el filtro de particulas que localiza contra ese mapa.
- capturas/: capturas de RViz mostrando la localizacion (entregable Parte 2)

CONFIG AMCL:
- base_frame_id=base_footprint (coincide con el frame del EKF)
- robot_model_type=DifferentialMotionModel (robot diferencial)
- set_initial_pose=true con la pose del spawn (x=1.3044, y=-7.2093,
  yaw=1.5708): arranca localizado sin el boton de RViz
- Sin bond_timeout:0.0 porque map_server y amcl son de Nav2 y hablan bond

FIX GEOMETRIA (mobile_base.xacro):
- Colision del castor: radius 0.01 -> 0.0145 (la rueda mide 29mm diametro).
  La esfera chica hacia cabecear al robot e inclinaba el LIDAR. Corregido,
  quedo horizontal. Critico para AMCL y el costmap de Parte 3.

SETUP:
- setup.py: entrada data_files para instalar maps/ (sin esto map_server no
  encuentra el mapa)

File: my_robot_description/urdf/mobile_base.xacro (robot description, xacro)
@@ -147,5 +147,5 @@
       <origin xyz="0 0 0" rpy="0 0 0"/>
       <geometry>
-        <sphere radius="0.01"/>
+        <sphere radius="0.0145"/>
       </geometry>
     </collision>
